File: board/board.kicad_sch (KiCad schematic)
At the start: 15 parts, among them J1 RAHMB20AUETR, J2 PINHD_1x2_Male, SW1 B3F-1002, SW2 B3F-1002, SW3 B3F-1002, SW4 B3F-1002, U1 ESP32-S3-WROOM-1-N16R8, U2 MCP73831T-2DCI_MC, U3 TPS74533PCQWDRVRQ1, U4 MAX17048G_T10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

Commit message: add gerbers and BOM
Parts:
- J2, L1: now left out of the parts list
- LED1: DigiKey_Part_Number (none) -> 568-16347CT-ND
- SW1, SW2, SW3, SW4: DigiKey_Part_Number (none) -> SW401-ND
- U1: DigiKey_Part_Number (none) -> 5407-ESP32-S3-WROOM-1-N16R8CT-ND
- U3: DigiKey_Part_Number (none) -> 296-TPS74533PCQWDRVRQ1CT-ND; MANUFACTURER (none) -> TI(德州仪器); Manufacturer TI(德州仪器) -> (none)
- U5: DigiKey_Part_Number (none) -> 785-1000-1-ND
Changed lines of the file:
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@@
+			)
+		)
+		(property "DigiKey_Part_Number" "5407-ESP32-S3-WROOM-1-N16R8CT-ND "
+			(at 44.45 35.56 0)
+			(hide yes)
+			(show_name no)
+			(do_not_autoplace no)
+			(effects
+				(font
+					(size 1.27 1.27)
+				)
 			)
 		)
@@
 			)
 		)
+		(property "DigiKey_Part_Number" "  SW401-ND"
+			(at 222.25 153.67 0)
+			(hide yes)
+			(show_name no)
+			(do_not_autoplace no)
+			(effects
+				(font
+					(size 1.27 1.27)
+				)
+			)
+		)
 		(pin "3"
 		)
@@
 			)
 		)
-		(property "Manufacturer" "TI(德州仪器)"
+		(property "MANUFACTURER" "TI(德州仪器)"
 			(at 82.55 168.91 0)
 			(hide yes)
@@
 		(property "LCSC Part" "C2860924"
 			(at 82.55 173.99 0)
+			(hide yes)
+			(show_name no)
+			(do_not_autoplace no)
+			(effects
+				(font
+					(size 1.27 1.27)
+				)
+			)
+		)
+		(property "DigiKey_Part_Number" "296-TPS74533PCQWDRVRQ1CT-ND "
+			(at 82.55 152.4 0)
 			(hide yes)
 			(show_name no)
@@
 			)
 		)
+		(property "DigiKey_Part_Number" "568-16347CT-ND"
+			(at 129.54 119.38 0)
+			(hide yes)
+			(show_name no)
+			(do_not_autoplace no)
+			(effects
+				(font
+					(size 1.27 1.27)
+				)
+			)
+		)
 		(pin "1"
 		)
@@
 			)
 		)
+		(property "DigiKey_Part_Number" "  SW401-ND"
+			(at 222.25 133.35 0)
+			(hide yes)
+			(show_name no)
+			(do_not_autoplace no)
+			(effects
+				(font
+					(size 1.27 1.27)
+				)
+			)
+		)
 		(pin "3"
 		)
@@
 		(body_style 1)
 		(exclude_from_sim no)
-		(in_bom yes)
+		(in_bom no)
 		(on_board yes)
 		(in_pos_files yes)
@@
 			)
 		)
+		(property "DigiKey_Part_Number" "  SW401-ND"
+			(at 142.24 44.45 0)
+			(hide yes)
+			(show_name no)
+			(do_not_autoplace no)
+			(effects
+				(font
+					(size 1.27 1.27)
+				)
+			)
+		)
 		(pin "3"
 		)
@@
 			)
 		)
+		(property "DigiKey_Part_Number" "785-1000-1-ND"
+			(at 129.54 100.33 0)
+			(hide yes)
+			(show_name no)
+			(do_not_autoplace no)
+			(effects
+				(font
+					(size 1.27 1.27)
+				)
+			)
+		)
 		(pin "1"
 		)
@@
 		(body_style 1)
 		(exclude_from_sim no)
-		(in_bom yes)
+		(in_bom no)
 		(on_board yes)
 		(in_pos_files yes)
@@
 			(at 222.25 113.03 0)
 			(hide yes)
+			(show_name no)
+			(do_not_autoplace no)
+			(effects
+				(font
+					(size 1.27 1.27)
+				)
+			)
+		)
+		(property "DigiKey_Part_Number" "  SW401-ND"
+			(at 222.25 113.03 0)
+			(hide yes)
